File: CustomPlexi/Boost.kicad_sch (KiCad schematic)
At the start: 8 parts, among them U1 TL074

Commit message: Signal chain ok except separated volumes
Parts:
- C8, C9: footprint Capacitor_SMD:C_0603_1608Metric_Pad1.08x0.95mm_HandSolder -> Capacitor_SMD_AKL:C_0603_1608Metric
- R10, R11, R8, R9: footprint Resistor_SMD:R_0603_1608Metric_Pad0.98x0.95mm_HandSolder -> Resistor_SMD_AKL:R_0603_1608Metric
Changed lines of the file:
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@@
       (effects (font (size 1.27 1.27)))
     )
-    (property "Footprint" "Capacitor_SMD:C_0603_1608Metric_Pad1.08x0.95mm_HandSolder" (at 133.35 93.0148 0)
+    (property "Footprint" "Capacitor_SMD_AKL:C_0603_1608Metric" (at 133.35 93.0148 0)
       (effects (font (size 1.27 1.27)) hide)
     )
@@
       (effects (font (size 1.27 1.27)))
     )
-    (property "Footprint" "Resistor_SMD:R_0603_1608Metric_Pad0.98x0.95mm_HandSolder" (at 146.05 93.98 0)
+    (property "Footprint" "Resistor_SMD_AKL:R_0603_1608Metric" (at 146.05 93.98 0)
       (effects (font (size 1.27 1.27)) hide)
     )
@@
       (effects (font (size 1.27 1.27)) (justify right))
     )
-    (property "Footprint" "Resistor_SMD:R_0603_1608Metric_Pad0.98x0.95mm_HandSolder" (at 116.84 76.2 0)
+    (property "Footprint" "Resistor_SMD_AKL:R_0603_1608Metric" (at 116.84 76.2 0)
       (effects (font (size 1.27 1.27)) hide)
     )
@@
       (effects (font (size 1.27 1.27)))
     )
-    (property "Footprint" "Capacitor_SMD:C_0603_1608Metric_Pad1.08x0.95mm_HandSolder" (at 110.744 101.9048 0)
+    (property "Footprint" "Capacitor_SMD_AKL:C_0603_1608Metric" (at 110.744 101.9048 0)
       (effects (font (size 1.27 1.27)) hide)
     )
@@
       (effects (font (size 1.27 1.27)) (justify right))
     )
-    (property "Footprint" "Resistor_SMD:R_0603_1608Metric_Pad0.98x0.95mm_HandSolder" (at 167.894 88.9 0)
+    (property "Footprint" "Resistor_SMD_AKL:R_0603_1608Metric" (at 167.894 88.9 0)
       (effects (font (size 1.27 1.27)) hide)
     )
@@
       (effects (font (size 1.27 1.27)))
     )
-    (property "Footprint" "Resistor_SMD:R_0603_1608Metric_Pad0.98x0.95mm_HandSolder" (at 106.68 102.87 0)
-      (effects (font (size 1.27 1.27)) hide)
-    )
+    (property "Footprint" "Resistor_SMD_AKL:R_0603_1608Metric" (at 106.68 102.87 0)
+      (effects (font (size 1.27 1.27)) hide)
+    )

Commit message: some changes
Parts:
- added D17: LD271, LED_THT:LED_D5.0mm_IRGrey, symbol LED:LD271
- added R3: 100k, Resistor_SMD_AKL:R_0603_1608Metric, symbol PCM_Resistor_AKL:R_0603
- added SW1: Boost Enable/Disable, symbol Switch:SW_Push_DPDT
Connections:
- net GND: now also D17.1 (K)
- net at C9.2, R10.2, U1.8: now also SW1.2 (B)
- net SW_Boost_Off renamed Boost
- net Boost: now also SW1.3 (C)
- net SW_Boost_On: no longer names the net of RV5.1
- net SW_Boost_On: now also SW1.1 (A)
- new net: R3.1, SW1.4 (A)
- new net: D17.2 (A), R3.2
- new net +9V: SW1.5 (B)
Other:
- moved on the sheet: C9, R10, R11, R9, RV5

Commit message: switches reviewed
Parts:
- removed D17: LD271, LED_THT:LED_D5.0mm_IRGrey, symbol LED:LD271
- removed R3: 100k, Resistor_SMD_AKL:R_0603_1608Metric, symbol PCM_Resistor_AKL:R_0603
- removed SW1: Boost Enable/Disable, symbol Switch:SW_Push_DPDT
- added SW7: Boost Enable/Disable, symbol CustomLib:SW_SPDT_x2
Connections:
- net Boost: now also SW7.1
- net at C9.2, R10.2, U1.8: now also SW7.2
- net at RV5.1: now also SW7.3
- net Boost_In renamed Tone_Out/Boost_In
Changed lines of the file:
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@@
-    (stroke (width 0) (type default))
-  )
-  (wire (pts (xy 130.81 64.77) (xy 135.89 64.77))
-    (stroke (width 0) (type default))
-  )
-  (wire (pts (xy 110.49 64.77) (xy 123.19 64.77))
-    (stroke (width 0) (type default))
-  )
-  (wire (pts (xy 110.49 73.66) (xy 110.49 74.93))
     (stroke (width 0) (type default))
   )
@@
     (stroke (width 0) (type default))
   )
-  (wire (pts (xy 148.59 62.23) (xy 148.59 60.96))
-    (stroke (width 0) (type default))
-  )
   (wire (pts (xy 153.67 93.98) (xy 157.48 93.98))
     (stroke (width 0) (type default))
@@
     (stroke (width 0) (type default))
   )
-  (wire (pts (xy 110.49 66.04) (xy 110.49 64.77))
-    (stroke (width 0) (type default))
-  )
   (wire (pts (xy 110.744 102.87) (xy 116.84 102.87))
     (stroke (width 0) (type default))
   )
   (wire (pts (xy 127 69.85) (xy 135.89 69.85))
-    (stroke (width 0) (type default))
-  )
-  (wire (pts (xy 146.05 62.23) (xy 148.59 62.23))
     (stroke (width 0) (type default))
   )
@@
     (effects (font (size 1.27 1.27)) (justify left bottom))
   )
-  (global_label "Boost_In" (shape input) (at 72.39 102.87 180) (fields_autoplaced)
+  (global_label "Tone_Out{slash}Boost_In" (shape input) (at 72.39 102.87 180) (fields_autoplaced)
     (effects (font (size 1.27 1.27)) (justify right))
-    (property "Intersheetrefs" "${INTERSHEET_REFS}" (at 61.441 102.87 0)
+    (property "Intersheetrefs" "${INTERSHEET_REFS}" (at 51.5835 102.87 0)
       (effects (font (size 1.27 1.27)) (justify right) hide)
     )
@@
     )
   )
-  (symbol (lib_id "PCM_Resistor_AKL:R_0603") (at 127 64.77 270) (unit 1)
-    (in_bom yes) (on_board yes) (dnp no)
-    (property "Reference" "R3" (at 127 59.69 90)
-      (effects (font (size 1.27 1.27)))
-    )
-    (property "Value" "100k" (at 127 62.23 90)
-      (effects (font (size 1.27 1.27)))
-    )
-    (property "Footprint" "Resistor_SMD_AKL:R_0603_1608Metric" (at 115.57 64.77 0)
-      (effects (font (size 1.27 1.27)) hide)
-    )
-    (property "Datasheet" "~" (at 127 64.77 0)
-      (effects (font (size 1.27 1.27)) hide)
-    )
-    (pin "1")
-    (pin "2")
-    (instances
-      (project "CustomPlexi"
-        (path "/cb47f45c-6a2b-402e-a3a9-bf4992e06e45"
-          (reference "R3") (unit 1)
-        )
-        (path "/cb47f45c-6a2b-402e-a3a9-bf4992e06e45/bb03f90a-acf2-4514-8da0-ce840f9be904"
-          (reference "R8") (unit 1)
-        )
-        (path "/cb47f45c-6a2b-402e-a3a9-bf4992e06e45/46194796-04b4-4b0f-a843-2a3656b84ab8"
-          (reference "R3") (unit 1)
-        )
-        (path "/cb47f45c-6a2b-402e-a3a9-bf4992e06e45/b3a3e8ef-e747-456f-8933-4bcf39be44f4"
-          (reference "R16") (unit 1)
-        )
-        (path "/cb47f45c-6a2b-402e-a3a9-bf4992e06e45/456125fd-895a-4d81-aa0f-bb315183acbb"
-          (reference "R16") (unit 1)
-        )
-      )
-    )
-  )
   (symbol (lib_id "Device:R_Potentiometer") (at 127 74.93 270) (mirror x) (unit 1)
     (in_bom yes) (on_board yes) (dnp no)
@@
     )
   )
-  (symbol (lib_id "power:GND") (at 110.49 74.93 0) (unit 1)
-    (in_bom yes) (on_board yes) (dnp no) (fields_autoplaced)
-    (property "Reference" "#PWR01" (at 110.49 81.28 0)
-      (effects (font (size 1.27 1.27)) hide)
-    )
-    (property "Value" "GND" (at 110.49 80.01 0)
-      (effects (font (size 1.27 1.27)))
-    )
-    (property "Footprint" "" (at 110.49 74.93 0)
-      (effects (font (size 1.27 1.27)) hide)
-    )
-    (property "Datasheet" "" (at 110.49 74.93 0)
-      (effects (font (size 1.27 1.27)) hide)
-    )
-    (pin "1")
-    (instances
-      (project "CustomPlexi"
-        (path "/cb47f45c-6a2b-402e-a3a9-bf4992e06e45"
-          (reference "#PWR01") (unit 1)
-        )
-        (path "/cb47f45c-6a2b-402e-a3a9-bf4992e06e45/9b0d4c7f-a409-4743-8b6f-6499ab699d39"
-          (reference "#PWR03") (unit 1)
-        )
-        (path "/cb47f45c-6a2b-402e-a3a9-bf4992e06e45/46194796-04b4-4b0f-a843-2a3656b84ab8"
-          (reference "#PWR06") (unit 1)
-        )
-        (path "/cb47f45c-6a2b-402e-a3a9-bf4992e06e45/b3a3e8ef-e747-456f-8933-4bcf39be44f4"
-          (reference "#PWR013") (unit 1)
-        )
-        (path "/cb47f45c-6a2b-402e-a3a9-bf4992e06e45/456125fd-895a-4d81-aa0f-bb315183acbb"
-          (reference "#PWR015") (unit 1)
+  (symbol (lib_id "CustomLib:SW_SPDT_x2") (at 140.97 72.39 0) (mirror y) (unit 1)
+    (in_bom yes) (on_board yes) (dnp no)
+    (property "Reference" "SW7" (at 140.97 64.77 0)
+      (effects (font (size 1.27 1.27)))
+    )
+    (property "Value" "Boost Enable/Disable" (at 140.97 67.31 0)
+      (effects (font (size 1.27 1.27)))
+    )
+    (property "Footprint" "" (at 139.7 67.31 0)
+      (effects (font (size 1.27 1.27)) hide)
+    )
+    (property "Datasheet" "" (at 139.7 67.31 0)
+      (effects (font (size 1.27 1.27)) hide)
+    )
+    (pin "1")
+    (pin "2")
+    (pin "3")
+    (pin "1")
+    (pin "2")
+    (pin "3")
+    (instances
+      (project "CustomPlexi"
+        (path "/cb47f45c-6a2b-402e-a3a9-bf4992e06e45/456125fd-895a-4d81-aa0f-bb315183acbb"
+          (reference "SW7") (unit 1)
         )
       )
@@
         (path "/cb47f45c-6a2b-402e-a3a9-bf4992e06e45/456125fd-895a-4d81-aa0f-bb315183acbb"
           (reference "#PWR08") (unit 1)
-        )
-      )
-    )
-  )
-  (symbol (lib_id "power:+9V") (at 148.59 60.96 0) (unit 1)
-    (in_bom yes) (on_board yes) (dnp no) (fields_autoplaced)
-    (property "Reference" "#PWR015" (at 148.59 64.77 0)
-      (effects (font (size 1.27 1.27)) hide)
-    )
-    (property "Value" "+9V" (at 148.59 57.15 0)
-      (effects (font (size 1.27 1.27)))
-    )
-    (property "Footprint" "" (at 148.59 60.96 0)
-      (effects (font (size 1.27 1.27)) hide)
-    )
-    (property "Datasheet" "" (at 148.59 60.96 0)
-      (effects (font (size 1.27 1.27)) hide)
-    )
-    (pin "1")
-    (instances
-      (project "CustomPlexi"
-        (path "/cb47f45c-6a2b-402e-a3a9-bf4992e06e45/b3a3e8ef-e747-456f-8933-4bcf39be44f4"
-          (reference "#PWR015") (unit 1)
-        )
-        (path "/cb47f45c-6a2b-402e-a3a9-bf4992e06e45/456125fd-895a-4d81-aa0f-bb315183acbb"
-          (reference "#PWR013") (unit 1)
-        )
-      )
-    )
-  )
-  (symbol (lib_id "Switch:SW_Push_DPDT") (at 140.97 67.31 180) (unit 1)
-    (in_bom yes) (on_board yes) (dnp no)
-    (property "Reference" "SW1" (at 140.97 81.28 0)
-      (effects (font (size 1.27 1.27)))
-    )
-    (property "Value" "Boost Enable/Disable" (at 140.97 78.74 0)
-      (effects (font (size 1.27 1.27)))
-    )
-    (property "Footprint" "" (at 140.97 72.39 0)
-      (effects (font (size 1.27 1.27)) hide)
-    )
-    (property "Datasheet" "~" (at 140.97 72.39 0)
-      (effects (font (size 1.27 1.27)) hide)
-    )
-    (pin "1")
-    (pin "2")
-    (pin "3")
-    (pin "4")
-    (pin "5")
-    (pin "6")
-    (instances
-      (project "CustomPlexi"
-        (path "/cb47f45c-6a2b-402e-a3a9-bf4992e06e45"
-          (reference "SW1") (unit 1)
-        )
-        (path "/cb47f45c-6a2b-402e-a3a9-bf4992e06e45/b3a3e8ef-e747-456f-8933-4bcf39be44f4"
-          (reference "SW5") (unit 1)
-        )
-        (path "/cb47f45c-6a2b-402e-a3a9-bf4992e06e45/456125fd-895a-4d81-aa0f-bb315183acbb"
-          (reference "SW3") (unit 1)
         )
       )
@@
         )
       )
-    )
-  )
-  (symbol (lib_id "LED:LD271") (at 110.49 68.58 270) (mirror x) (unit 1)
-    (in_bom yes) (on_board yes) (dnp no)
-    (property "Reference" "D17" (at 107.95 69.088 90)
-      (effects (font (size 1.27 1.27)) (justify right))
-    )
-    (property "Value" "LD271" (at 107.95 71.628 90)
-      (effects (font (size 1.27 1.27)) (justify right))
-    )
-    (property "Footprint" "LED_THT:LED_D5.0mm_IRGrey" (at 114.935 68.58 0)
-      (effects (font (size 1.27 1.27)) hide)
-    )
-    (property "Datasheet" "http://www.alliedelec.com/m/d/40788c34903a719969df15f1fbea1056.pdf" (at 110.49 69.85 0)
-      (effects (font (size 1.27 1.27)) hide)
-    )
-    (pin "1")
-    (pin "2")
-    (instances
-      (project "CustomPlexi"
-        (path "/cb47f45c-6a2b-402e-a3a9-bf4992e06e45/b3a3e8ef-e747-456f-8933-4bcf39be44f4"
-          (reference "D17") (unit 1)
-        )
-        (path "/cb47f45c-6a2b-402e-a3a9-bf4992e06e45/456125fd-895a-4d81-aa0f-bb315183acbb"
-          (reference "D17") (unit 1)
-        )
-      )

Commit message: commit
Parts:
- added J1: Conn_01x02_Pin, Connector_PinHeader_2.54mm:PinHeader_1x02_P2.54mm_Vertical, symbol Connector:Conn_01x02_Pin
- C8, C9: footprint Capacitor_SMD_AKL:C_0603_1608Metric -> Capacitor_SMD:C_0402_1005Metric_Pad0.74x0.62mm_HandSolder
- R10, R11, R8, R9: footprint Resistor_SMD_AKL:R_0603_1608Metric -> Resistor_SMD:R_0402_1005Metric_Pad0.72x0.64mm_HandSolder
- RV5: footprint (none) -> PCM_Potentiometer_THT_US_AKL_Double:Potentiometer_Vishay_148-149_Single_Vertical
- SW7: footprint (none) -> CustomLib:SW_SPST_x2_PinHeader2.54mm
- U1: footprint (none) -> Package_SO:SOIC-14W_7.5x9mm_P1.27mm
Connections:
- net GND: now also J1.2 (Pin_2)
- net To_Amp: now also J1.1 (Pin_1)
Changed lines of the file:
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@@
   (junction (at 138.43 93.98) (diameter 0) (color 0 0 0 0)
   )
+  (junction (at 187.96 93.98) (diameter 0) (color 0 0 0 0)
+  )
   (wire (pts (xy 72.39 102.87) (xy 91.44 102.87))
     (stroke (width 0) (type default))
@@
     (stroke (width 0) (type default))
   )
+  (wire (pts (xy 187.96 87.63) (xy 199.39 87.63))
+    (stroke (width 0) (type default))
+  )
   (wire (pts (xy 130.81 74.93) (xy 135.89 74.93))
     (stroke (width 0) (type default))
@@
     (stroke (width 0) (type default))
   )
-  (wire (pts (xy 171.704 93.98) (xy 181.61 93.98))
+  (wire (pts (xy 171.704 93.98) (xy 187.96 93.98))
     (stroke (width 0) (type default))
   )
@@
     (stroke (width 0) (type default))
   )
+  (wire (pts (xy 187.96 96.52) (xy 187.96 100.33))
+    (stroke (width 0) (type default))
+  )
   (wire (pts (xy 171.704 93.98) (xy 171.704 96.52))
     (stroke (width 0) (type default))
@@
   )
   (wire (pts (xy 127 69.85) (xy 135.89 69.85))
+    (stroke (width 0) (type default))
+  )
+  (wire (pts (xy 187.96 87.63) (xy 187.96 93.98))
     (stroke (width 0) (type default))
   )
@@
     )
   )
-  (global_label "To_Amp" (shape output) (at 181.61 93.98 0) (fields_autoplaced)
+  (global_label "To_Amp" (shape output) (at 199.39 87.63 0) (fields_autoplaced)
     (effects (font (size 1.27 1.27)) (justify left))
-    (property "Intersheetrefs" "${INTERSHEET_REFS}" (at 191.5309 93.98 0)
+    (property "Intersheetrefs" "${INTERSHEET_REFS}" (at 209.3109 87.63 0)
       (effects (font (size 1.27 1.27)) (justify left) hide)
     )
@@
       (effects (font (size 1.27 1.27)))
     )
-    (property "Footprint" "Capacitor_SMD_AKL:C_0603_1608Metric" (at 132.08 93.0148 0)
+    (property "Footprint" "Capacitor_SMD:C_0402_1005Metric_Pad0.74x0.62mm_HandSolder" (at 132.08 93.0148 0)
       (effects (font (size 1.27 1.27)) hide)
     )
@@
       (effects (font (size 1.27 1.27)))
     )
-    (property "Footprint" "Resistor_SMD_AKL:R_0603_1608Metric" (at 149.86 93.98 0)
+    (property "Footprint" "Resistor_SMD:R_0402_1005Metric_Pad0.72x0.64mm_HandSolder" (at 149.86 93.98 0)
       (effects (font (size 1.27 1.27)) hide)
     )
@@
       (effects (font (size 1.27 1.27)) (justify right))
     )
-    (property "Footprint" "" (at 127 74.93 0)
+    (property "Footprint" "PCM_Potentiometer_THT_US_AKL_Double:Potentiometer_Vishay_148-149_Single_Vertical" (at 127 74.93 0)
       (effects (font (size 1.27 1.27)) hide)
     )
@@
         (path "/cb47f45c-6a2b-402e-a3a9-bf4992e06e45/456125fd-895a-4d81-aa0f-bb315183acbb"
           (reference "RV6") (unit 1)
+        )
+      )
+    )
+  )
+  (symbol (lib_id "Connector:Conn_01x02_Pin") (at 193.04 93.98 0) (mirror y) (unit 1)
+    (in_bom yes) (on_board yes) (dnp no)
+    (property "Reference" "J1" (at 194.31 95.885 0)
+      (effects (font (size 1.27 1.27)) (justify right))
+    )
+    (property "Value" "Conn_01x02_Pin" (at 194.31 93.345 0)
+      (effects (font (size 1.27 1.27)) (justify right))
+    )
+    (property "Footprint" "Connector_PinHeader_2.54mm:PinHeader_1x02_P2.54mm_Vertical" (at 193.04 93.98 0)
+      (effects (font (size 1.27 1.27)) hide)
+    )
+    (property "Datasheet" "~" (at 193.04 93.98 0)
+      (effects (font (size 1.27 1.27)) hide)
+    )
+    (pin "1")
+    (pin "2")
+    (instances
+      (project "CustomPlexi"
+        (path "/cb47f45c-6a2b-402e-a3a9-bf4992e06e45/c4a7bcdf-70be-4e6d-b7b4-c53de8d52358"
+          (reference "J1") (unit 1)
+        )
+        (path "/cb47f45c-6a2b-402e-a3a9-bf4992e06e45/9b0d4c7f-a409-4743-8b6f-6499ab699d39"
+          (reference "J2") (unit 1)
+        )
+        (path "/cb47f45c-6a2b-402e-a3a9-bf4992e06e45/456125fd-895a-4d81-aa0f-bb315183acbb"
+          (reference "J3") (unit 1)
         )
       )
@@
       (effects (font (size 1.27 1.27)))
     )
-    (property "Footprint" "" (at 139.7 67.31 0)
+    (property "Footprint" "CustomLib:SW_SPST_x2_PinHeader2.54mm" (at 139.7 67.31 0)
       (effects (font (size 1.27 1.27)) hide)
     )
@@
       (effects (font (size 1.27 1.27)) (justify right))
     )
-    (property "Footprint" "Resistor_SMD_AKL:R_0603_1608Metric" (at 116.84 74.93 0)
+    (property "Footprint" "Resistor_SMD:R_0402_1005Metric_Pad0.72x0.64mm_HandSolder" (at 116.84 74.93 0)
       (effects (font (size 1.27 1.27)) hide)
     )
@@
       (effects (font (size 1.27 1.27)))
     )
-    (property "Footprint" "" (at 127 107.95 0)
+    (property "Footprint" "Package_SO:SOIC-14W_7.5x9mm_P1.27mm" (at 127 107.95 0)
       (effects (font (size 1.27 1.27)) hide)
     )
@@
       (effects (font (size 1.27 1.27)))
     )
-    (property "Footprint" "Capacitor_SMD_AKL:C_0603_1608Metric" (at 110.744 101.9048 0)
+    (property "Footprint" "Capacitor_SMD:C_0402_1005Metric_Pad0.74x0.62mm_HandSolder" (at 110.744 101.9048 0)
       (effects (font (size 1.27 1.27)) hide)
     )
@@
       (effects (font (size 1.27 1.27)) (justify right))
     )
-    (property "Footprint" "Resistor_SMD_AKL:R_0603_1608Metric" (at 171.704 88.9 0)
+    (property "Footprint" "Resistor_SMD:R_0402_1005Metric_Pad0.72x0.64mm_HandSolder" (at 171.704 88.9 0)
       (effects (font (size 1.27 1.27)) hide)
     )
@@
       (effects (font (size 1.27 1.27)))
     )
-    (property "Footprint" "Resistor_SMD_AKL:R_0603_1608Metric" (at 106.68 102.87 0)
+    (property "Footprint" "Resistor_SMD:R_0402_1005Metric_Pad0.72x0.64mm_HandSolder" (at 106.68 102.87 0)
       (effects (font (size 1.27 1.27)) hide)
     )
@@
         )
       )
+    )
+  )
+  (symbol (lib_id "power:GND") (at 187.96 100.33 0) (unit 1)
+    (in_bom yes) (on_board yes) (dnp no) (fields_autoplaced)
+    (property "Reference" "#PWR04" (at 187.96 106.68 0)
+      (effects (font (size 1.27 1.27)) hide)
+    )
+    (property "Value" "GND" (at 187.96 105.41 0)
+      (effects (font (size 1.27 1.27)))
+    )
+    (property "Footprint" "" (at 187.96 100.33 0)
+      (effects (font (size 1.27 1.27)) hide)
+    )
+    (property "Datasheet" "" (at 187.96 100.33 0)
+      (effects (font (size 1.27 1.27)) hide)
+    )
+    (pin "1")
+    (instances
+      (project "CustomPlexi"
+        (path "/cb47f45c-6a2b-402e-a3a9-bf4992e06e45"
+          (reference "#PWR04") (unit 1)
+        )
+        (path "/cb47f45c-6a2b-402e-a3a9-bf4992e06e45/456125fd-895a-4d81-aa0f-bb315183acbb"
+          (reference "#PWR030") (unit 1)
+        )
+      )
