File: CustomPlexi/InputFIlterPlusBuffer.kicad_sch (KiCad schematic)
At the start: 5 parts, among them U1 TL074

Commit message: Signal chain ok except separated volumes
Parts:
- C1, C2: footprint Capacitor_SMD:C_0603_1608Metric_Pad1.08x0.95mm_HandSolder -> Capacitor_SMD_AKL:C_0603_1608Metric
- R1, R2: footprint Resistor_SMD:R_0603_1608Metric_Pad0.98x0.95mm_HandSolder -> Resistor_SMD_AKL:R_0603_1608Metric
Connections:
- net Buffer_Out/Plexi_In renamed Buffer_Out
Changed lines of the file:
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@@
     (stroke (width 0) (type default))
   )
-  (global_label "Buffer_Out{slash}Plexi_In" (shape output) (at 143.51 62.23 0) (fields_autoplaced)
+  (global_label "Buffer_Out" (shape output) (at 143.51 62.23 0) (fields_autoplaced)
     (effects (font (size 1.27 1.27)) (justify left))
-    (property "Intersheetrefs" "${INTERSHEET_REFS}" (at 165.0424 62.23 0)
+    (property "Intersheetrefs" "${INTERSHEET_REFS}" (at 156.3338 62.23 0)
       (effects (font (size 1.27 1.27)) (justify left) hide)
     )
@@
       (effects (font (size 1.27 1.27)) (justify right))
     )
-    (property "Footprint" "Resistor_SMD:R_0603_1608Metric_Pad0.98x0.95mm_HandSolder" (at 92.71 59.69 0)
+    (property "Footprint" "Resistor_SMD_AKL:R_0603_1608Metric" (at 92.71 59.69 0)
       (effects (font (size 1.27 1.27)) hide)
     )
@@
       (effects (font (size 1.27 1.27)))
     )
-    (property "Footprint" "Capacitor_SMD:C_0603_1608Metric_Pad1.08x0.95mm_HandSolder" (at 90.17 63.8048 0)
+    (property "Footprint" "Capacitor_SMD_AKL:C_0603_1608Metric" (at 90.17 63.8048 0)
       (effects (font (size 1.27 1.27)) hide)
     )
@@
       (effects (font (size 1.27 1.27)))
     )
-    (property "Footprint" "Resistor_SMD:R_0603_1608Metric_Pad0.98x0.95mm_HandSolder" (at 78.74 64.77 0)
+    (property "Footprint" "Resistor_SMD_AKL:R_0603_1608Metric" (at 78.74 64.77 0)
       (effects (font (size 1.27 1.27)) hide)
     )
@@
       (effects (font (size 1.27 1.27)) (justify left))
     )
-    (property "Footprint" "Capacitor_SMD:C_0603_1608Metric_Pad1.08x0.95mm_HandSolder" (at 80.9752 74.93 0)
+    (property "Footprint" "Capacitor_SMD_AKL:C_0603_1608Metric" (at 80.9752 74.93 0)
       (effects (font (size 1.27 1.27)) hide)
     )

Commit message: switches reviewed
Connections:
- net Buffer_Out renamed Buffer_Out/Preamp_In
Changed lines of the file:
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@@
     (stroke (width 0) (type default))
   )
-  (global_label "Buffer_Out" (shape output) (at 143.51 62.23 0) (fields_autoplaced)
+  (global_label "Buffer_Out{slash}Preamp_In" (shape output) (at 143.51 62.23 0) (fields_autoplaced)
     (effects (font (size 1.27 1.27)) (justify left))
-    (property "Intersheetrefs" "${INTERSHEET_REFS}" (at 156.3338 62.23 0)
+    (property "Intersheetrefs" "${INTERSHEET_REFS}" (at 167.5218 62.23 0)
       (effects (font (size 1.27 1.27)) (justify left) hide)
     )

Commit message: commit
Parts:
- added J1: Conn_01x02_Pin, Connector_PinHeader_2.54mm:PinHeader_1x02_P2.54mm_Vertical, symbol Connector:Conn_01x02_Pin
- C1, C2: footprint Capacitor_SMD_AKL:C_0603_1608Metric -> Capacitor_SMD:C_0402_1005Metric_Pad0.74x0.62mm_HandSolder
- R1, R2: footprint Resistor_SMD_AKL:R_0603_1608Metric -> Resistor_SMD:R_0402_1005Metric_Pad0.72x0.64mm_HandSolder
- U1: footprint (none) -> Package_SO:SOIC-14W_7.5x9mm_P1.27mm
Connections:
- net GND: now also J1.2 (Pin_2)
- net Guitar_In: now also J1.1 (Pin_1)
Changed lines of the file:
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@@
   (junction (at 124.46 62.23) (diameter 0) (color 0 0 0 0)
   )
+  (junction (at 53.34 64.77) (diameter 0) (color 0 0 0 0)
+  )
   (junction (at 80.01 77.47) (diameter 0) (color 0 0 0 0)
   )
@@
     (stroke (width 0) (type default))
   )
+  (wire (pts (xy 53.34 67.31) (xy 53.34 71.12))
+    (stroke (width 0) (type default))
+  )
   (wire (pts (xy 119.38 62.23) (xy 124.46 62.23))
     (stroke (width 0) (type default))
@@
     (stroke (width 0) (type default))
   )
+  (wire (pts (xy 53.34 64.77) (xy 63.5 64.77))
+    (stroke (width 0) (type default))
+  )
   (wire (pts (xy 80.01 77.47) (xy 92.71 77.47))
     (stroke (width 0) (type default))
@@
     (stroke (width 0) (type default))
   )
+  (wire (pts (xy 53.34 58.42) (xy 53.34 64.77))
+    (stroke (width 0) (type default))
+  )
   (wire (pts (xy 71.12 64.77) (xy 80.01 64.77))
     (stroke (width 0) (type default))
@@
     (stroke (width 0) (type default))
   )
-  (wire (pts (xy 54.61 64.77) (xy 63.5 64.77))
+  (wire (pts (xy 39.37 58.42) (xy 53.34 58.42))
     (stroke (width 0) (type default))
   )
@@
     )
   )
-  (global_label "Guitar_In" (shape input) (at 54.61 64.77 180) (fields_autoplaced)
+  (global_label "Guitar_In" (shape input) (at 39.37 58.42 180) (fields_autoplaced)
     (effects (font (size 1.27 1.27)) (justify right))
-    (property "Intersheetrefs" "${INTERSHEET_REFS}" (at 43.2981 64.77 0)
+    (property "Intersheetrefs" "${INTERSHEET_REFS}" (at 28.0581 58.42 0)
       (effects (font (size 1.27 1.27)) (justify right) hide)
     )
@@
       (effects (font (size 1.27 1.27)))
     )
-    (property "Footprint" "" (at 110.49 64.77 0)
+    (property "Footprint" "Package_SO:SOIC-14W_7.5x9mm_P1.27mm" (at 110.49 64.77 0)
       (effects (font (size 1.27 1.27)) hide)
     )
@@
       (effects (font (size 1.27 1.27)) (justify right))
     )
-    (property "Footprint" "Resistor_SMD_AKL:R_0603_1608Metric" (at 92.71 59.69 0)
+    (property "Footprint" "Resistor_SMD:R_0402_1005Metric_Pad0.72x0.64mm_HandSolder" (at 92.71 59.69 0)
       (effects (font (size 1.27 1.27)) hide)
     )
@@
     )
   )
+  (symbol (lib_id "Connector:Conn_01x02_Pin") (at 48.26 64.77 0) (unit 1)
+    (in_bom yes) (on_board yes) (dnp no) (fields_autoplaced)
+    (property "Reference" "J1" (at 48.895 60.96 0)
+      (effects (font (size 1.27 1.27)))
+    )
+    (property "Value" "Conn_01x02_Pin" (at 48.895 63.5 0)
+      (effects (font (size 1.27 1.27)))
+    )
+    (property "Footprint" "Connector_PinHeader_2.54mm:PinHeader_1x02_P2.54mm_Vertical" (at 48.26 64.77 0)
+      (effects (font (size 1.27 1.27)) hide)
+    )
+    (property "Datasheet" "~" (at 48.26 64.77 0)
+      (effects (font (size 1.27 1.27)) hide)
+    )
+    (pin "1")
+    (pin "2")
+    (instances
+      (project "CustomPlexi"
+        (path "/cb47f45c-6a2b-402e-a3a9-bf4992e06e45/c4a7bcdf-70be-4e6d-b7b4-c53de8d52358"
+          (reference "J1") (unit 1)
+        )
+        (path "/cb47f45c-6a2b-402e-a3a9-bf4992e06e45/9b0d4c7f-a409-4743-8b6f-6499ab699d39"
+          (reference "J2") (unit 1)
+        )
+      )
+    )
+  )
   (symbol (lib_id "PCM_Capacitor_AKL:C_0603") (at 86.36 64.77 90) (unit 1)
     (in_bom yes) (on_board yes) (dnp no) (fields_autoplaced)
@@
       (effects (font (size 1.27 1.27)))
     )
-    (property "Footprint" "Capacitor_SMD_AKL:C_0603_1608Metric" (at 90.17 63.8048 0)
+    (property "Footprint" "Capacitor_SMD:C_0402_1005Metric_Pad0.74x0.62mm_HandSolder" (at 90.17 63.8048 0)
       (effects (font (size 1.27 1.27)) hide)
     )
@@
     )
   )
+  (symbol (lib_id "power:GND") (at 53.34 71.12 0) (unit 1)
+    (in_bom yes) (on_board yes) (dnp no) (fields_autoplaced)
+    (property "Reference" "#PWR01" (at 53.34 77.47 0)
+      (effects (font (size 1.27 1.27)) hide)
+    )
+    (property "Value" "GND" (at 53.34 76.2 0)
+      (effects (font (size 1.27 1.27)))
+    )
+    (property "Footprint" "" (at 53.34 71.12 0)
+      (effects (font (size 1.27 1.27)) hide)
+    )
+    (property "Datasheet" "" (at 53.34 71.12 0)
+      (effects (font (size 1.27 1.27)) hide)
+    )
+    (pin "1")
+    (instances
+      (project "CustomPlexi"
+        (path "/cb47f45c-6a2b-402e-a3a9-bf4992e06e45"
+          (reference "#PWR01") (unit 1)
+        )
+        (path "/cb47f45c-6a2b-402e-a3a9-bf4992e06e45/9b0d4c7f-a409-4743-8b6f-6499ab699d39"
+          (reference "#PWR029") (unit 1)
+        )
+      )
+    )
+  )
   (symbol (lib_id "PCM_Resistor_AKL:R_0603") (at 67.31 64.77 90) (unit 1)
     (in_bom yes) (on_board yes) (dnp no) (fields_autoplaced)
@@
       (effects (font (size 1.27 1.27)))
     )
-    (property "Footprint" "Resistor_SMD_AKL:R_0603_1608Metric" (at 78.74 64.77 0)
+    (property "Footprint" "Resistor_SMD:R_0402_1005Metric_Pad0.72x0.64mm_HandSolder" (at 78.74 64.77 0)
       (effects (font (size 1.27 1.27)) hide)
     )
@@
       (effects (font (size 1.27 1.27)) (justify left))
     )
-    (property "Footprint" "Capacitor_SMD_AKL:C_0603_1608Metric" (at 80.9752 74.93 0)
-      (effects (font (size 1.27 1.27)) hide)
-    )
+    (property "Footprint" "Capacitor_SMD:C_0402_1005Metric_Pad0.74x0.62mm_HandSolder" (at 80.9752 74.93 0)
+      (effects (font (size 1.27 1.27)) hide)
+    )
