File: CustomPlexi/Leds.kicad_sch (KiCad schematic)
At the start: 11 parts, among them SW4 Pedal Enable, SW5 Plexi Channel Select, SW8 Preamp Enable

Commit message: switches reviewed
Parts:
- added D17: LD271, LED_THT:LED_D5.0mm_IRGrey, symbol LED:LD271
- added R3: 100k, Resistor_SMD_AKL:R_0603_1608Metric, symbol PCM_Resistor_AKL:R_0603
- added SW7: Boost Enable/Disable, symbol CustomLib:SW_SPDT_x2
Connections:
- net +9V: now also SW7.2
- net GND: now also D17.1 (K)
- new net: D17.2 (A), R3.2
- new net: R3.1, SW7.1

Commit message: commit
Parts:
- R3: footprint Resistor_SMD_AKL:R_0603_1608Metric -> Resistor_SMD:R_0402_1005Metric_Pad0.72x0.64mm_HandSolder
- SW4, SW8: footprint (none) -> CustomLib:SW_SPST_x3_PinHeader2.54mm
- SW5: footprint (none) -> CustomLib:SW_SPST_x4_PinHeader2.54mm
- SW7: footprint (none) -> CustomLib:SW_SPST_x2_PinHeader2.54mm
Changed lines of the file:
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@@
       (effects (font (size 1.27 1.27)))
     )
-    (property "Footprint" "Resistor_SMD_AKL:R_0603_1608Metric" (at 132.08 63.5 0)
+    (property "Footprint" "Resistor_SMD:R_0402_1005Metric_Pad0.72x0.64mm_HandSolder" (at 132.08 63.5 0)
       (effects (font (size 1.27 1.27)) hide)
     )
@@
       (effects (font (size 1.27 1.27)))
     )
-    (property "Footprint" "Resistor_SMD_AKL:R_0603_1608Metric" (at 93.98 63.5 0)
+    (property "Footprint" "Resistor_SMD:R_0402_1005Metric_Pad0.72x0.64mm_HandSolder" (at 93.98 63.5 0)
       (effects (font (size 1.27 1.27)) hide)
     )
@@
       (effects (font (size 1.27 1.27)))
     )
-    (property "Footprint" "" (at 121.92 39.37 0)
+    (property "Footprint" "CustomLib:SW_SPST_x4_PinHeader2.54mm" (at 121.92 39.37 0)
       (effects (font (size 1.27 1.27)) hide)
     )
@@
       (effects (font (size 1.27 1.27)))
     )
-    (property "Footprint" "Resistor_SMD_AKL:R_0603_1608Metric" (at 144.78 63.5 0)
+    (property "Footprint" "Resistor_SMD:R_0402_1005Metric_Pad0.72x0.64mm_HandSolder" (at 144.78 63.5 0)
       (effects (font (size 1.27 1.27)) hide)
     )
@@
       (effects (font (size 1.27 1.27)))
     )
-    (property "Footprint" "Resistor_SMD_AKL:R_0603_1608Metric" (at 55.88 63.5 0)
+    (property "Footprint" "Resistor_SMD:R_0402_1005Metric_Pad0.72x0.64mm_HandSolder" (at 55.88 63.5 0)
       (effects (font (size 1.27 1.27)) hide)
     )
@@
       (effects (font (size 1.27 1.27)))
     )
-    (property "Footprint" "" (at 45.72 39.37 0)
+    (property "Footprint" "CustomLib:SW_SPST_x3_PinHeader2.54mm" (at 45.72 39.37 0)
       (effects (font (size 1.27 1.27)) hide)
     )
@@
       (effects (font (size 1.27 1.27)))
     )
-    (property "Footprint" "" (at 175.26 39.37 0)
+    (property "Footprint" "CustomLib:SW_SPST_x2_PinHeader2.54mm" (at 175.26 39.37 0)
       (effects (font (size 1.27 1.27)) hide)
     )
@@
         )
         (path "/cb47f45c-6a2b-402e-a3a9-bf4992e06e45/b3a3e8ef-e747-456f-8933-4bcf39be44f4"
-          (reference "SW3") (unit 2)
+          (reference "SW7") (unit 2)
         )
       )
@@
       (effects (font (size 1.27 1.27)))
     )
-    (property "Footprint" "" (at 81.28 39.37 0)
+    (property "Footprint" "CustomLib:SW_SPST_x3_PinHeader2.54mm" (at 81.28 39.37 0)
       (effects (font (size 1.27 1.27)) hide)
     )
@@
       (effects (font (size 1.27 1.27)))
     )
-    (property "Footprint" "Resistor_SMD_AKL:R_0603_1608Metric" (at 190.5 63.5 0)
-      (effects (font (size 1.27 1.27)) hide)
-    )
+    (property "Footprint" "Resistor_SMD:R_0402_1005Metric_Pad0.72x0.64mm_HandSolder" (at 190.5 63.5 0)
+      (effects (font (size 1.27 1.27)) hide)
+    )

Commit message: changed refdes
Parts:
- renumbered D19 to D18, D18 to D19, D17 to D20
Changed lines of the file:
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@@
         )
         (path "/cb47f45c-6a2b-402e-a3a9-bf4992e06e45/b3a3e8ef-e747-456f-8933-4bcf39be44f4"
-          (reference "#PWR012") (unit 1)
+          (reference "#PWR027") (unit 1)
         )
       )
@@
         )
         (path "/cb47f45c-6a2b-402e-a3a9-bf4992e06e45/b3a3e8ef-e747-456f-8933-4bcf39be44f4"
-          (reference "#PWR011") (unit 1)
+          (reference "#PWR026") (unit 1)
         )
       )
@@
         )
         (path "/cb47f45c-6a2b-402e-a3a9-bf4992e06e45/b3a3e8ef-e747-456f-8933-4bcf39be44f4"
-          (reference "R18") (unit 1)
+          (reference "R21") (unit 1)
         )
       )
@@
         )
         (path "/cb47f45c-6a2b-402e-a3a9-bf4992e06e45/b3a3e8ef-e747-456f-8933-4bcf39be44f4"
-          (reference "#PWR015") (unit 1)
+          (reference "#PWR032") (unit 1)
         )
         (path "/cb47f45c-6a2b-402e-a3a9-bf4992e06e45/456125fd-895a-4d81-aa0f-bb315183acbb"
@@
         )
         (path "/cb47f45c-6a2b-402e-a3a9-bf4992e06e45/b3a3e8ef-e747-456f-8933-4bcf39be44f4"
-          (reference "#PWR017") (unit 1)
+          (reference "#PWR030") (unit 1)
         )
       )
@@
   (symbol (lib_id "LED:LD271") (at 190.5 60.96 270) (mirror x) (unit 1)
     (in_bom yes) (on_board yes) (dnp no)
-    (property "Reference" "D17" (at 187.96 61.468 90)
+    (property "Reference" "D20" (at 187.96 61.468 90)
       (effects (font (size 1.27 1.27)) (justify right))
     )
@@
       (project "CustomPlexi"
         (path "/cb47f45c-6a2b-402e-a3a9-bf4992e06e45/b3a3e8ef-e747-456f-8933-4bcf39be44f4"
-          (reference "D17") (unit 1)
+          (reference "D20") (unit 1)
         )
         (path "/cb47f45c-6a2b-402e-a3a9-bf4992e06e45/456125fd-895a-4d81-aa0f-bb315183acbb"
@@
         )
         (path "/cb47f45c-6a2b-402e-a3a9-bf4992e06e45/b3a3e8ef-e747-456f-8933-4bcf39be44f4"
-          (reference "R4") (unit 1)
+          (reference "R20") (unit 1)
         )
       )
@@
         )
         (path "/cb47f45c-6a2b-402e-a3a9-bf4992e06e45/b3a3e8ef-e747-456f-8933-4bcf39be44f4"
-          (reference "R17") (unit 1)
+          (reference "R22") (unit 1)
         )
       )
@@
         )
         (path "/cb47f45c-6a2b-402e-a3a9-bf4992e06e45/b3a3e8ef-e747-456f-8933-4bcf39be44f4"
-          (reference "D15") (unit 1)
+          (reference "D17") (unit 1)
         )
       )
@@
         )
         (path "/cb47f45c-6a2b-402e-a3a9-bf4992e06e45/b3a3e8ef-e747-456f-8933-4bcf39be44f4"
-          (reference "R11") (unit 1)
+          (reference "R19") (unit 1)
         )
       )
@@
   (symbol (lib_id "LED:LD271") (at 132.08 59.69 90) (unit 1)
     (in_bom yes) (on_board yes) (dnp no) (fields_autoplaced)
-    (property "Reference" "D19" (at 134.62 60.198 90)
+    (property "Reference" "D18" (at 134.62 60.198 90)
       (effects (font (size 1.27 1.27)) (justify right))
     )
@@
       (project "CustomPlexi"
         (path "/cb47f45c-6a2b-402e-a3a9-bf4992e06e45/b3a3e8ef-e747-456f-8933-4bcf39be44f4"
-          (reference "D19") (unit 1)
+          (reference "D18") (unit 1)
         )
       )
@@
         )
         (path "/cb47f45c-6a2b-402e-a3a9-bf4992e06e45/b3a3e8ef-e747-456f-8933-4bcf39be44f4"
-          (reference "SW4") (unit 3)
+          (reference "SW1") (unit 3)
         )
       )
@@
         )
         (path "/cb47f45c-6a2b-402e-a3a9-bf4992e06e45/b3a3e8ef-e747-456f-8933-4bcf39be44f4"
-          (reference "#PWR014") (unit 1)
+          (reference "#PWR028") (unit 1)
         )
       )
@@
         )
         (path "/cb47f45c-6a2b-402e-a3a9-bf4992e06e45/b3a3e8ef-e747-456f-8933-4bcf39be44f4"
-          (reference "SW6") (unit 3)
+          (reference "SW3") (unit 3)
         )
       )
@@
   (symbol (lib_id "power:+9V") (at 109.22 41.91 0) (unit 1)
     (in_bom yes) (on_board yes) (dnp no) (fields_autoplaced)
-    (property "Reference" "#PWR016" (at 109.22 45.72 0)
+    (property "Reference" "#PWR029" (at 109.22 45.72 0)
       (effects (font (size 1.27 1.27)) hide)
     )
@@
       (project "CustomPlexi"
         (path "/cb47f45c-6a2b-402e-a3a9-bf4992e06e45/b3a3e8ef-e747-456f-8933-4bcf39be44f4"
-          (reference "#PWR016") (unit 1)
+          (reference "#PWR029") (unit 1)
         )
       )
@@
   (symbol (lib_id "LED:LD271") (at 144.78 59.69 90) (unit 1)
     (in_bom yes) (on_board yes) (dnp no) (fields_autoplaced)
-    (property "Reference" "D18" (at 147.32 60.198 90)
+    (property "Reference" "D19" (at 147.32 60.198 90)
       (effects (font (size 1.27 1.27)) (justify right))
     )
@@
       (project "CustomPlexi"
         (path "/cb47f45c-6a2b-402e-a3a9-bf4992e06e45/b3a3e8ef-e747-456f-8933-4bcf39be44f4"
-          (reference "D18") (unit 1)
+          (reference "D19") (unit 1)
         )
       )
@@
   (symbol (lib_id "power:+9V") (at 160.02 43.18 0) (unit 1)
     (in_bom yes) (on_board yes) (dnp no) (fields_autoplaced)
-    (property "Reference" "#PWR013" (at 160.02 46.99 0)
+    (property "Reference" "#PWR031" (at 160.02 46.99 0)
       (effects (font (size 1.27 1.27)) hide)
     )
@@
       (project "CustomPlexi"
         (path "/cb47f45c-6a2b-402e-a3a9-bf4992e06e45/b3a3e8ef-e747-456f-8933-4bcf39be44f4"
-          (reference "#PWR013") (unit 1)
+          (reference "#PWR031") (unit 1)
         )
         (path "/cb47f45c-6a2b-402e-a3a9-bf4992e06e45/456125fd-895a-4d81-aa0f-bb315183acbb"
@@
   (symbol (lib_id "power:+9V") (at 31.75 43.18 0) (unit 1)
     (in_bom yes) (on_board yes) (dnp no) (fields_autoplaced)
-    (property "Reference" "#PWR010" (at 31.75 46.99 0)
+    (property "Reference" "#PWR025" (at 31.75 46.99 0)
       (effects (font (size 1.27 1.27)) hide)
     )
@@
       (project "CustomPlexi"
         (path "/cb47f45c-6a2b-402e-a3a9-bf4992e06e45/b3a3e8ef-e747-456f-8933-4bcf39be44f4"
-          (reference "#PWR010") (unit 1)
+          (reference "#PWR025") (unit 1)
         )
       )
@@
         )
         (path "/cb47f45c-6a2b-402e-a3a9-bf4992e06e45/b3a3e8ef-e747-456f-8933-4bcf39be44f4"
-          (reference "R16") (unit 1)
+          (reference "R23") (unit 1)
         )
         (path "/cb47f45c-6a2b-402e-a3a9-bf4992e06e45/456125fd-895a-4d81-aa0f-bb315183acbb"
