File: CustomPlexi/preamp.kicad_sch (KiCad schematic)
At the start: 10 parts, among them U1 TL074

Commit message: switches reviewed
Parts:
- added SW4: Pedal Enable, symbol CustomLib:SW_SPDT_x3
- added SW6, SW8: Preamp Enable, symbol CustomLib:SW_SPDT_x3
Connections:
- net Preamp_Out/Plexi_In: now also SW6.2; no longer RV4.2
- net Preamp_In: no longer names the net of C3.1
- net Preamp_In: now also SW8.1
- new net: RV4.2, SW6.1
- new net: SW4.1, SW8.2
- new net: SW6.3, SW8.3
- new net Buffer_Out/Preamp_In: SW4.2
- new net Pedal_SC: SW4.3
Other:
- moved on the sheet: C3, D5, D6, R3, RV2, RV4, U1D

Commit message: commit
Parts:
- C3: footprint Capacitor_SMD_AKL:C_0603_1608Metric -> Capacitor_SMD:C_0402_1005Metric_Pad0.74x0.62mm_HandSolder
- R3: footprint Resistor_SMD_AKL:R_0603_1608Metric -> Resistor_SMD:R_0402_1005Metric_Pad0.72x0.64mm_HandSolder
- RV2, RV4: footprint (none) -> PCM_Potentiometer_THT_US_AKL_Double:Potentiometer_Vishay_148-149_Single_Vertical
- SW4, SW6, SW8: footprint (none) -> CustomLib:SW_SPST_x3_PinHeader2.54mm
- U1: footprint (none) -> Package_SO:SOIC-14W_7.5x9mm_P1.27mm
Connections:
- net PreAmp_Volume: now reaches RV4.2, SW6.1
- net PreAmp renamed PreAmp_Gain
Other:
- moved on the sheet: SW6B
Changed lines of the file:
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@@
     (stroke (width 0) (type default))
   )
-  (wire (pts (xy 118.11 121.92) (xy 196.85 121.92))
+  (wire (pts (xy 118.11 121.92) (xy 200.66 121.92))
     (stroke (width 0) (type default))
   )
@@
     (stroke (width 0) (type default))
   )
-  (wire (pts (xy 196.85 121.92) (xy 196.85 109.22))
+  (wire (pts (xy 200.66 121.92) (xy 200.66 109.22))
     (stroke (width 0) (type default))
   )
@@
     (stroke (width 0) (type default))
   )
-  (wire (pts (xy 180.34 104.14) (xy 196.85 104.14))
+  (wire (pts (xy 180.34 104.14) (xy 200.66 104.14))
     (stroke (width 0) (type default))
   )
@@
     (stroke (width 0) (type default))
   )
-  (wire (pts (xy 207.01 106.68) (xy 218.44 106.68))
+  (wire (pts (xy 210.82 106.68) (xy 218.44 106.68))
     (stroke (width 0) (type default))
   )
@@
     (stroke (width 0) (type default))
   )
-  (label "PreAmp" (at 161.29 63.5 0) (fields_autoplaced)
+  (label "PreAmp_Volume" (at 181.61 104.14 0) (fields_autoplaced)
+    (effects (font (size 1.27 1.27)) (justify left bottom))
+  )
+  (label "PreAmp_Gain" (at 161.29 63.5 0) (fields_autoplaced)
     (effects (font (size 1.27 1.27)) (justify left bottom))
   )
@@
       (effects (font (size 1.27 1.27)))
     )
-    (property "Footprint" "" (at 154.94 99.06 0)
+    (property "Footprint" "Package_SO:SOIC-14W_7.5x9mm_P1.27mm" (at 154.94 99.06 0)
       (effects (font (size 1.27 1.27)) hide)
     )
@@
       (effects (font (size 1.27 1.27)))
     )
-    (property "Footprint" "Capacitor_SMD_AKL:C_0603_1608Metric" (at 139.7 98.0948 0)
+    (property "Footprint" "Capacitor_SMD:C_0402_1005Metric_Pad0.74x0.62mm_HandSolder" (at 139.7 98.0948 0)
       (effects (font (size 1.27 1.27)) hide)
     )
@@
       (effects (font (size 1.27 1.27)) (justify right))
     )
-    (property "Footprint" "" (at 176.53 104.14 0)
+    (property "Footprint" "PCM_Potentiometer_THT_US_AKL_Double:Potentiometer_Vishay_148-149_Single_Vertical" (at 176.53 104.14 0)
       (effects (font (size 1.27 1.27)) hide)
     )
@@
       (effects (font (size 1.27 1.27)))
     )
-    (property "Footprint" "Resistor_SMD_AKL:R_0603_1608Metric" (at 114.3 58.42 0)
+    (property "Footprint" "Resistor_SMD:R_0402_1005Metric_Pad0.72x0.64mm_HandSolder" (at 114.3 58.42 0)
       (effects (font (size 1.27 1.27)) hide)
     )
@@
       (effects (font (size 1.27 1.27)))
     )
-    (property "Footprint" "" (at 114.3 96.52 0)
+    (property "Footprint" "CustomLib:SW_SPST_x3_PinHeader2.54mm" (at 114.3 96.52 0)
       (effects (font (size 1.27 1.27)) hide)
     )
@@
       (effects (font (size 1.27 1.27)))
     )
-    (property "Footprint" "" (at 160.02 58.42 0)
+    (property "Footprint" "PCM_Potentiometer_THT_US_AKL_Double:Potentiometer_Vishay_148-149_Single_Vertical" (at 160.02 58.42 0)
       (effects (font (size 1.27 1.27)) hide)
     )
@@
       (effects (font (size 1.27 1.27)))
     )
-    (property "Footprint" "" (at 88.9 99.06 0)
+    (property "Footprint" "CustomLib:SW_SPST_x3_PinHeader2.54mm" (at 88.9 99.06 0)
       (effects (font (size 1.27 1.27)) hide)
     )
@@
       (effects (font (size 1.27 1.27)))
     )
-    (property "Footprint" "Resistor_SMD_AKL:R_0603_1608Metric" (at 138.43 58.42 0)
+    (property "Footprint" "Resistor_SMD:R_0402_1005Metric_Pad0.72x0.64mm_HandSolder" (at 138.43 58.42 0)
       (effects (font (size 1.27 1.27)) hide)
     )
@@
       (effects (font (size 1.27 1.27)))
     )
-    (property "Footprint" "Capacitor_SMD_AKL:C_0603_1608Metric" (at 139.7 57.4548 0)
+    (property "Footprint" "Capacitor_SMD:C_0402_1005Metric_Pad0.74x0.62mm_HandSolder" (at 139.7 57.4548 0)
       (effects (font (size 1.27 1.27)) hide)
     )
@@
       (effects (font (size 1.27 1.27)))
     )
-    (property "Footprint" "Capacitor_SMD_AKL:C_0603_1608Metric" (at 158.75 85.3948 0)
+    (property "Footprint" "Capacitor_SMD:C_0402_1005Metric_Pad0.74x0.62mm_HandSolder" (at 158.75 85.3948 0)
       (effects (font (size 1.27 1.27)) hide)
     )
@@
     )
   )
-  (symbol (lib_id "CustomLib:SW_SPDT_x3") (at 201.93 106.68 0) (mirror y) (unit 2)
-    (in_bom yes) (on_board yes) (dnp no)
-    (property "Reference" "SW6" (at 201.93 99.06 0)
-      (effects (font (size 1.27 1.27)))
-    )
-    (property "Value" "Preamp Enable" (at 201.93 101.6 0)
-      (effects (font (size 1.27 1.27)))
-    )
-    (property "Footprint" "" (at 200.66 101.6 0)
-      (effects (font (size 1.27 1.27)) hide)
-    )
-    (property "Datasheet" "" (at 200.66 101.6 0)
-      (effects (font (size 1.27 1.27)) hide)
-    )
+  (symbol (lib_id "CustomLib:SW_SPDT_x3") (at 205.74 106.68 0) (mirror y) (unit 2)
+    (in_bom yes) (on_board yes) (dnp no)
+    (property "Reference" "SW6" (at 205.74 99.06 0)
+      (effects (font (size 1.27 1.27)))
+    )
+    (property "Value" "Preamp Enable" (at 205.74 101.6 0)
+      (effects (font (size 1.27 1.27)))
+    )
+    (property "Footprint" "CustomLib:SW_SPST_x3_PinHeader2.54mm" (at 204.47 101.6 0)
+      (effects (font (size 1.27 1.27)) hide)
+    )
+    (property "Datasheet" "" (at 204.47 101.6 0)
+      (effects (font (size 1.27 1.27)) hide)
+    )

Commit message: deleted tone stack
Parts:
- removed U1: TL074, Package_SO:SOIC-14W_7.5x9mm_P1.27mm, symbol Amplifier_Operational:TL074
Changed lines of the file:
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@@
-    )
-  )
-  (symbol (lib_id "Amplifier_Operational:TL074") (at 156.21 96.52 0) (mirror x) (unit 4)
-    (in_bom yes) (on_board yes) (dnp no)
-    (property "Reference" "U1" (at 156.21 105.41 0)
-      (effects (font (size 1.27 1.27)))
-    )
-    (property "Value" "TL074" (at 156.21 102.87 0)
-      (effects (font (size 1.27 1.27)))
-    )
-    (property "Footprint" "Package_SO:SOIC-14W_7.5x9mm_P1.27mm" (at 154.94 99.06 0)
-      (effects (font (size 1.27 1.27)) hide)
-    )
-    (property "Datasheet" "http://www.ti.com/lit/ds/symlink/tl071.pdf" (at 157.48 101.6 0)
-      (effects (font (size 1.27 1.27)) hide)
-    )
-    (pin "1")
-    (pin "2")
-    (pin "3")
-    (pin "5")
-    (pin "6")
-    (pin "7")
-    (pin "10")
-    (pin "8")
-    (pin "9")
-    (pin "12")
-    (pin "13")
-    (pin "14")
-    (pin "11")
-    (pin "4")
-    (instances
-      (project "CustomPlexi"
-        (path "/cb47f45c-6a2b-402e-a3a9-bf4992e06e45"
-          (reference "U1") (unit 4)
-        )
-        (path "/cb47f45c-6a2b-402e-a3a9-bf4992e06e45/d67dc5e3-b5e6-4ced-a0aa-c1f6a7e7b9d1"
-          (reference "U2") (unit 4)
-        )
-        (path "/cb47f45c-6a2b-402e-a3a9-bf4992e06e45/46194796-04b4-4b0f-a843-2a3656b84ab8"
-          (reference "U1") (unit 4)
-        )
-      )
     )
   )

Commit message: Full ts808
Parts:
- added C3: 220n, Capacitor_SMD:C_0402_1005Metric_Pad0.74x0.62mm_HandSolder, symbol PCM_Capacitor_AKL:C_0603
- added C3: 200n, Capacitor_SMD:C_0402_1005Metric_Pad0.74x0.62mm_HandSolder, symbol PCM_Capacitor_AKL:C_0603
- added C3: 1u, Capacitor_SMD:C_0402_1005Metric_Pad0.74x0.62mm_HandSolder, symbol PCM_Capacitor_AKL:C_0603
- added R3 (x3): 1k, Resistor_SMD:R_0402_1005Metric_Pad0.72x0.64mm_HandSolder, symbol PCM_Resistor_AKL:R_0603
- added R3: 220, Resistor_SMD:R_0402_1005Metric_Pad0.72x0.64mm_HandSolder, symbol PCM_Resistor_AKL:R_0603
- added RV2: 20k Lin, PCM_Potentiometer_THT_US_AKL_Double:Potentiometer_Vishay_148-149_Single_Vertical, symbol Device:R_Potentiometer
- added U5: RC4558, symbol Amplifier_Operational:RC4558
- C3: value 4.7k -> 47n
- R3: value 51k -> 4.7k
- SW8: value Preamp Enable -> TS_Enable
Connections:
- net GND: now also C3.1, R3.2
- net at C3.1, C3.2, D5.2 (A)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: now also U5.2 (-)
- net at C3.2: now also U5.3 (+)
- net PreAmp_Gain renamed TS_Gain
- net TS_Gain: now also R3.2, U5.1; no longer RV4.1
- net PreAmp_Volume renamed TS_Volume
- new net: C3.1, R3.1 (x2)
- new net: R3.2, RV4.1
- new net: C3.2, R3.1, RV2.3, U5.5 (+)
- new net: R3.2, RV2.1, U5.6 (-)
- new net: C3.2, R3.1, U5.7
- new net TS_Tone: C3.2, RV2.2
Other:
- moved on the sheet: C3, D5, D6, R3, RV2, RV4, SW4A, SW6B, SW8A

Commit message: changed refdes
Parts:
- renumbered D6 to D1, D5 to D2, SW4 to SW1, SW8 to SW2, SW6 to SW3, U5 to U2
Other:
- moved on the sheet: SW1A
Changed lines of the file:
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@@
   (junction (at 101.6 87.63) (diameter 0) (color 0 0 0 0)
   )
-  (wire (pts (xy 57.15 107.95) (xy 57.15 134.62))
+  (wire (pts (xy 63.5 107.95) (xy 63.5 134.62))
     (stroke (width 0) (type default))
   )
@@
     (stroke (width 0) (type default))
   )
-  (wire (pts (xy 57.15 102.87) (xy 72.39 102.87))
+  (wire (pts (xy 63.5 102.87) (xy 72.39 102.87))
     (stroke (width 0) (type default))
   )
@@
     (stroke (width 0) (type default))
   )
-  (wire (pts (xy 57.15 134.62) (xy 182.88 134.62))
+  (wire (pts (xy 63.5 134.62) (xy 182.88 134.62))
     (stroke (width 0) (type default))
   )
@@
     (stroke (width 0) (type default))
   )
-  (wire (pts (xy 40.64 105.41) (xy 46.99 105.41))
+  (wire (pts (xy 46.99 105.41) (xy 53.34 105.41))
     (stroke (width 0) (type default))
   )
@@
     (effects (font (size 1.27 1.27)) (justify left bottom))
   )
-  (global_label "Buffer_Out{slash}Preamp_In" (shape input) (at 40.64 105.41 180) (fields_autoplaced)
+  (global_label "Buffer_Out{slash}Preamp_In" (shape input) (at 46.99 105.41 180) (fields_autoplaced)
     (effects (font (size 1.27 1.27)) (justify right))
-    (property "Intersheetrefs" "${INTERSHEET_REFS}" (at 16.6282 105.41 0)
+    (property "Intersheetrefs" "${INTERSHEET_REFS}" (at 22.9782 105.41 0)
       (effects (font (size 1.27 1.27)) (justify right) hide)
     )
@@
         )
         (path "/cb47f45c-6a2b-402e-a3a9-bf4992e06e45/46194796-04b4-4b0f-a843-2a3656b84ab8"
-          (reference "R23") (unit 1)
+          (reference "R8") (unit 1)
         )
       )
@@
   (symbol (lib_id "Diode:1N4148") (at 113.03 78.74 0) (mirror y) (unit 1)
     (in_bom yes) (on_board yes) (dnp no)
-    (property "Reference" "D5" (at 113.03 73.66 0)
+    (property "Reference" "D2" (at 113.03 73.66 0)
       (effects (font (size 1.27 1.27)))
     )
@@
       (project "CustomPlexi"
         (path "/cb47f45c-6a2b-402e-a3a9-bf4992e06e45/46194796-04b4-4b0f-a843-2a3656b84ab8"
-          (reference "D5") (unit 1)
+          (reference "D2") (unit 1)
         )
       )
@@
         )
         (path "/cb47f45c-6a2b-402e-a3a9-bf4992e06e45/46194796-04b4-4b0f-a843-2a3656b84ab8"
-          (reference "C1") (unit 1)
+          (reference "C4") (unit 1)
         )
       )
@@
         )
         (path "/cb47f45c-6a2b-402e-a3a9-bf4992e06e45/46194796-04b4-4b0f-a843-2a3656b84ab8"
-          (reference "#PWR031") (unit 1)
+          (reference "#PWR05") (unit 1)
         )
       )
@@
         )
         (path "/cb47f45c-6a2b-402e-a3a9-bf4992e06e45/46194796-04b4-4b0f-a843-2a3656b84ab8"
-          (reference "RV9") (unit 1)
+          (reference "RV3") (unit 1)
         )
       )
@@
   (symbol (lib_id "Amplifier_Operational:RC4558") (at 114.3 97.79 0) (mirror x) (unit 1)
     (in_bom yes) (on_board yes) (dnp no)
-    (property "Reference" "U5" (at 114.3 106.68 0)
+    (property "Reference" "U2" (at 114.3 106.68 0)
       (effects (font (size 1.27 1.27)))
     )
@@
       (project "CustomPlexi"
         (path "/cb47f45c-6a2b-402e-a3a9-bf4992e06e45/46194796-04b4-4b0f-a843-2a3656b84ab8"
-          (reference "U5") (unit 1)
+          (reference "U2") (unit 1)
         )
       )
@@
   (symbol (lib_id "Amplifier_Operational:RC4558") (at 167.64 95.25 0) (mirror x) (unit 2)
     (in_bom yes) (on_board yes) (dnp no)
-    (property "Reference" "U5" (at 167.64 104.14 0)
+    (property "Reference" "U2" (at 167.64 104.14 0)
       (effects (font (size 1.27 1.27)))
     )
@@
       (project "CustomPlexi"
         (path "/cb47f45c-6a2b-402e-a3a9-bf4992e06e45/46194796-04b4-4b0f-a843-2a3656b84ab8"
-          (reference "U5") (unit 2)
+          (reference "U2") (unit 2)
         )
       )
@@
         )
         (path "/cb47f45c-6a2b-402e-a3a9-bf4992e06e45/46194796-04b4-4b0f-a843-2a3656b84ab8"
-          (reference "C18") (unit 1)
+          (reference "C7") (unit 1)
         )
       )
@@
         )
         (path "/cb47f45c-6a2b-402e-a3a9-bf4992e06e45/46194796-04b4-4b0f-a843-2a3656b84ab8"
-          (reference "R22") (unit 1)
+          (reference "R6") (unit 1)
         )
       )
@@
   (symbol (lib_id "Diode:1N4148") (at 113.03 69.85 0) (unit 1)
     (in_bom yes) (on_board yes) (dnp no)
-    (property "Reference" "D6" (at 113.03 64.77 0)
+    (property "Reference" "D1" (at 113.03 64.77 0)
       (effects (font (size 1.27 1.27)))
     )
@@
       (project "CustomPlexi"
         (path "/cb47f45c-6a2b-402e-a3a9-bf4992e06e45/46194796-04b4-4b0f-a843-2a3656b84ab8"
-          (reference "D6") (unit 1)
+          (reference "D1") (unit 1)
         )
       )
@@
         )
         (path "/cb47f45c-6a2b-402e-a3a9-bf4992e06e45/46194796-04b4-4b0f-a843-2a3656b84ab8"
-          (reference "#PWR032") (unit 1)
+          (reference "#PWR04") (unit 1)
         )
       )
@@
   (symbol (lib_id "CustomLib:SW_SPDT_x3") (at 77.47 102.87 0) (unit 1)
     (in_bom yes) (on_board yes) (dnp no) (fields_autoplaced)
-    (property "Reference" "SW8" (at 77.47 96.52 0)
+    (property "Reference" "SW2" (at 77.47 96.52 0)
       (effects (font (size 1.27 1.27)))
     )
@@
       (project "CustomPlexi"
         (path "/cb47f45c-6a2b-402e-a3a9-bf4992e06e45/46194796-04b4-4b0f-a843-2a3656b84ab8"
-          (reference "SW8") (unit 1)
+          (reference "SW2") (unit 1)
         )
       )
@@
         )
         (path "/cb47f45c-6a2b-402e-a3a9-bf4992e06e45/46194796-04b4-4b0f-a843-2a3656b84ab8"
-          (reference "C13") (unit 1)
+          (reference "C6") (unit 1)
         )
       )
@@
         )
         (path "/cb47f45c-6a2b-402e-a3a9-bf4992e06e45/46194796-04b4-4b0f-a843-2a3656b84ab8"
-          (reference "C19") (unit 1)
+          (reference "C8") (unit 1)
         )
       )
@@
         )
         (path "/cb47f45c-6a2b-402e-a3a9-bf4992e06e45/46194796-04b4-4b0f-a843-2a3656b84ab8"
-          (reference "R21") (unit 1)
-        )
-      )
-    )
-  )
-  (symbol (lib_id "CustomLib:SW_SPDT_x3") (at 52.07 105.41 0) (unit 1)
-    (in_bom yes) (on_board yes) (dnp no) (fields_autoplaced)
-    (property "Reference" "SW4" (at 52.07 97.79 0)
-      (effects (font (size 1.27 1.27)))
-    )
-    (property "Value" "Pedal Enable" (at 52.07 100.33 0)
-      (effects (font (size 1.27 1.27)))
-    )
-    (property "Footprint" "CustomLib:SW_SPST_x3_PinHeader2.54mm" (at 53.34 100.33 0)
-      (effects (font (size 1.27 1.27)) hide)
-    )
-    (property "Datasheet" "" (at 53.34 100.33 0)
-      (effects (font (size 1.27 1.27)) hide)
-    )
-    (pin "1")
-    (pin "2")
-    (pin "3")
-    (pin "1")
-    (pin "2")
-    (pin "3")
-    (pin "1")
-    (pin "2")
-    (pin "3")
-    (instances
-      (project "CustomPlexi"
-        (path "/cb47f45c-6a2b-402e-a3a9-bf4992e06e45/46194796-04b4-4b0f-a843-2a3656b84ab8"
-          (reference "SW4") (unit 1)
+          (reference "R7") (unit 1)
+        )
+      )
+    )
+  )
+  (symbol (lib_id "CustomLib:SW_SPDT_x3") (at 58.42 105.41 0) (unit 1)
+    (in_bom yes) (on_board yes) (dnp no) (fields_autoplaced)
+    (property "Reference" "SW1" (at 58.42 97.79 0)
+      (effects (font (size 1.27 1.27)))
+    )
+    (property "Value" "Pedal Enable" (at 58.42 100.33 0)
+      (effects (font (size 1.27 1.27)))
+    )
+    (property "Footprint" "CustomLib:SW_SPST_x3_PinHeader2.54mm" (at 59.69 100.33 0)
+      (effects (font (size 1.27 1.27)) hide)
+    )
+    (property "Datasheet" "" (at 59.69 100.33 0)
+      (effects (font (size 1.27 1.27)) hide)
+    )
+    (pin "1")
+    (pin "2")
+    (pin "3")
+    (pin "1")
+    (pin "2")
+    (pin "3")
+    (pin "1")
+    (pin "2")
+    (pin "3")
+    (instances
+      (project "CustomPlexi"
+        (path "/cb47f45c-6a2b-402e-a3a9-bf4992e06e45/46194796-04b4-4b0f-a843-2a3656b84ab8"
+          (reference "SW1") (unit 1)
         )
       )
@@
         )
         (path "/cb47f45c-6a2b-402e-a3a9-bf4992e06e45/46194796-04b4-4b0f-a843-2a3656b84ab8"
-          (reference "R1") (unit 1)
+          (reference "R4") (unit 1)
         )
       )
@@
         )
         (path "/cb47f45c-6a2b-402e-a3a9-bf4992e06e45/46194796-04b4-4b0f-a843-2a3656b84ab8"
-          (reference "C9") (unit 1)
+          (reference "C3") (unit 1)
         )
       )
@@
         )
         (path "/cb47f45c-6a2b-402e-a3a9-bf4992e06e45/46194796-04b4-4b0f-a843-2a3656b84ab8"
-          (reference "C2") (unit 1)
+          (reference "C5") (unit 1)
         )
       )
@@
   (symbol (lib_id "CustomLib:SW_SPDT_x3") (at 241.3 107.95 0) (mirror y) (unit 2)
     (in_bom yes) (on_board yes) (dnp no)
-    (property "Reference" "SW6" (at 241.3 100.33 0)
+    (property "Reference" "SW3" (at 241.3 100.33 0)
       (effects (font (size 1.27 1.27)))
     )
@@
       (project "CustomPlexi"
         (path "/cb47f45c-6a2b-402e-a3a9-bf4992e06e45/46194796-04b4-4b0f-a843-2a3656b84ab8"
-          (reference "SW6") (unit 2)
+          (reference "SW3") (unit 2)
         )
       )
@@
         )
         (path "/cb47f45c-6a2b-402e-a3a9-bf4992e06e45/46194796-04b4-4b0f-a843-2a3656b84ab8"
-          (reference "RV4") (unit 1)
+          (reference "RV2") (unit 1)
         )
       )
@@
         )
         (path "/cb47f45c-6a2b-402e-a3a9-bf4992e06e45/46194796-04b4-4b0f-a843-2a3656b84ab8"
-          (reference "#PWR02") (unit 1)
+          (reference "#PWR03") (unit 1)
         )
       )
@@
         )
         (path "/cb47f45c-6a2b-402e-a3a9-bf4992e06e45/46194796-04b4-4b0f-a843-2a3656b84ab8"
-          (reference "R20") (unit 1)
-        )
-      )
+          (reference "R5") (unit 1)
+        )
+      )
